Commit message: Adding lidar to urdf and simulation

File: description/gazebo_control.xacro (robot description, xacro)
@@ -6,6 +6,6 @@
             <left_joint>left_wheel_joint</left_joint>
             <right_joint>right_wheel_joint</right_joint>
-            <wheel_separation>0.2</wheel_separation>
-            <wheel_diameter>0.065</wheel_diameter>
+            <wheel_separation>${distance_cir_roue*2}</wheel_separation>
+            <wheel_diameter>${diametre_roue}</wheel_diameter>
             <!-- Limits -->
             <max_wheel_torque>200</max_wheel_torque>

File: description/robot.urdf.xacro (robot description, xacro)
@@ -3,3 +3,4 @@
     <xacro:include filename="robot_core.xacro" />
     <xacro:include filename="gazebo_control.xacro"/>
+    <xacro:include filename="lidar.xacro"/>
 </robot>

File: description/robot_core.xacro (robot description, xacro)
@@ -11,4 +11,7 @@
         <color rgba="0.2 0.2 1 1"/>
     </material>
+    <material name="red">
+        <color rgba="1 0 0 1"/>
+    </material>
     <material name="black">
         <color rgba="0 0 0 1"/>
@@ -17,25 +20,30 @@
     </link>
     <!-- CHASSIS -->
+    <xacro:property name="longueur_robot" value="0.25" />
+    <xacro:property name="largeur_robot" value="0.15" />
+    <xacro:property name="hauteur_robot" value="0.084" />
+    <xacro:property name="distance_cir" value="0.07836" />
+    <xacro:property name="masse_robot" value="0.5" />
     <joint name="chassis_joint" type="fixed">
         <parent link="base_link"/>
         <child link="chassis"/>
-        <origin xyz="-0.07836 0 0"/>
+        <origin xyz="-${distance_cir} 0 0"/>
     </joint>
     <link name="chassis">
         <visual>
-            <origin xyz="0.125 0 0.042" rpy="0 0 0"/>
+            <origin xyz="${longueur_robot/2} 0 ${hauteur_robot/2}" rpy="0 0 0"/>
             <geometry>
-                <box size="0.25 0.15 0.084"/>
+                <box size="${longueur_robot} ${largeur_robot} ${hauteur_robot}"/>
             </geometry>
             <material name="white"/>
         </visual>
         <collision>
-            <origin xyz="0.125 0 0.042" rpy="0 0 0"/>
+            <origin xyz="${longueur_robot/2} 0 ${hauteur_robot/2}" rpy="0 0 0"/>
             <geometry>
-                <box size="0.25 0.15 0.084"/>
+                <box size="${longueur_robot} ${largeur_robot} ${hauteur_robot}"/>
             </geometry>
         </collision>
-        <xacro:inertial_box mass="0.5" x="0.25" y="0.15" z="0.084">
-            <origin xyz="0.125 0 0.042" rpy="0 0 0"/>
+        <xacro:inertial_box mass="${masse_robot}" x="${longueur_robot}" y="${largeur_robot}" z="${hauteur_robot}">
+            <origin xyz="${longueur_robot/2} 0 ${hauteur_robot/2}" rpy="0 0 0"/>
         </xacro:inertial_box>
     </link>
@@ -44,8 +52,12 @@
     </gazebo>
     <!-- LEFT WHEEL -->
+    <xacro:property name="distance_cir_roue" value="0.1" />
+    <xacro:property name="longueur_roue" value="0.03" />
+    <xacro:property name="diametre_roue" value="0.065" />
+    <xacro:property name="masse_roue" value="0.1" />
     <joint name="left_wheel_joint" type="continuous">
         <parent link="base_link"/>
         <child link="left_wheel"/>
-        <origin xyz="0 0.1 0" rpy="-${pi/2} 0 0"/>
+        <origin xyz="0 ${distance_cir_roue} 0" rpy="-${pi/2} 0 0"/>
         <axis xyz="0 0 1"/>
     </joint>
@@ -53,5 +65,5 @@
         <visual>
             <geometry>
-                <cylinder length="0.04" radius="0.0325" />
+                <cylinder length="${longueur_roue}" radius="${diametre_roue/2}" />
             </geometry>
             <material name="blue"/>
@@ -59,8 +71,8 @@
         <collision>
             <geometry>
-                <cylinder length="0.04" radius="0.0325" />
+                <cylinder length="${longueur_roue}" radius="${diametre_roue/2}" />
             </geometry>
         </collision>
-        <xacro:inertial_cylinder mass="0.1" length="0.04" radius="0.0325">
+        <xacro:inertial_cylinder mass="${masse_roue}" length="${longueur_roue}" radius="${diametre_roue/2}">
             <origin xyz="0 0 0" rpy="0 0 0"/>
         </xacro:inertial_cylinder>
@@ -73,5 +85,5 @@
         <parent link="base_link"/>
         <child link="right_wheel"/>
-        <origin xyz="0 -0.1 0" rpy="${pi/2} 0 0"/>
+        <origin xyz="0 -${distance_cir_roue} 0" rpy="${pi/2} 0 0"/>
         <axis xyz="0 0 -1"/>
     </joint>
@@ -79,5 +91,5 @@
         <visual>
             <geometry>
-                <cylinder length="0.04" radius="0.0325" />
+                <cylinder length="${longueur_roue}" radius="${diametre_roue/2}" />
             </geometry>
             <material name="blue"/>
@@ -85,8 +97,8 @@
         <collision>
             <geometry>
-                <cylinder length="0.04" radius="0.0325" />
+                <cylinder length="${longueur_roue}" radius="${diametre_roue/2}" />
             </geometry>
         </collision>
-        <xacro:inertial_cylinder mass="0.1" length="0.04" radius="0.0325">
+        <xacro:inertial_cylinder mass="${masse_roue}" length="${longueur_roue}" radius="${diametre_roue/2}">
             <origin xyz="0 0 0" rpy="0 0 0"/>
         </xacro:inertial_cylinder>
@@ -96,13 +108,16 @@
     </gazebo>
     <!-- CASTER WHEEL -->
+    <xacro:property name="diametre_caster" value="${diametre_roue}" />
+    <xacro:property name="distance_caster" value="0.225" />
+    <xacro:property name="masse_caster" value="0.1" />
     <joint name="caster_wheel_joint" type="fixed">
         <parent link="chassis"/>
         <child link="caster_wheel"/>
-        <origin xyz="0.225 0 0" rpy="0 0 0"/>
+        <origin xyz="${distance_caster} 0 0" rpy="0 0 0"/>
     </joint>
     <link name="caster_wheel">
         <visual>
             <geometry>
-                <sphere radius="0.025" />
+                <sphere radius="${diametre_caster/2}" />
             </geometry>
             <material name="black"/>
@@ -110,8 +125,8 @@
         <collision>
             <geometry>
-                <sphere radius="0.025" />
+                <sphere radius="${diametre_caster/2}" />
             </geometry>
         </collision>
-        <xacro:inertial_sphere mass="0.1" radius="0.025">
+        <xacro:inertial_sphere mass="${masse_caster}" radius="${diametre_caster/2}">
             <origin xyz="0 0 0" rpy="0 0 0"/>
         </xacro:inertial_sphere>
