Commit message: Adding a camera to urdf and simulation

File: description/lidar.xacro (robot description, xacro)
@@ -30,5 +30,5 @@
         <sensor name="laser" type="ray">
             <pose> 0 0 0 0 0 0 </pose>
-            <visualize>true</visualize>
+            <visualize>false</visualize>  <!-- true if I want to see the blue lines -->
             <update_rate>10</update_rate>
             <ray>

File: description/robot.urdf.xacro (robot description, xacro)
@@ -4,4 +4,5 @@
     <!-- <xacro:include filename="gazebo_control.xacro"/> -->
     <xacro:include filename="lidar.xacro"/>
+    <xacro:include filename="camera.xacro"/>
     <xacro:include filename="ros2_control.xacro"/>
 </robot>

File: description/robot_core.xacro (robot description, xacro)
@@ -109,5 +109,5 @@
     <!-- CASTER WHEEL -->
     <xacro:property name="diametre_caster" value="${diametre_roue}" />
-    <xacro:property name="distance_caster" value="0.225" />
+    <xacro:property name="distance_caster" value="0.20" />
     <xacro:property name="masse_caster" value="0.1" />
     <joint name="caster_wheel_joint" type="fixed">
