Commit message: Simulation in gazebo

File: description/robot_core.xacro (robot description, xacro)
@@ -40,4 +40,7 @@
         </xacro:inertial_box>
     </link>
+    <gazebo reference="chassis">
+        <material>Gazebo/White</material>
+    </gazebo>
     <!-- LEFT WHEEL -->
     <joint name="left_wheel_joint" type="continuous">
@@ -63,4 +66,7 @@
         </xacro:inertial_cylinder>
     </link>
+    <gazebo reference="left_wheel">
+        <material>Gazebo/Blue</material>
+    </gazebo>
     <!-- RIGHT WHEEL -->
     <joint name="right_wheel_joint" type="continuous">
@@ -86,4 +92,7 @@
         </xacro:inertial_cylinder>
     </link>
+    <gazebo reference="right_wheel">
+        <material>Gazebo/Blue</material>
+    </gazebo>
     <!-- CASTER WHEEL -->
     <joint name="caster_wheel_joint" type="fixed">
@@ -108,3 +117,8 @@
         </xacro:inertial_sphere>
     </link>
+    <gazebo reference="caster_wheel">
+        <material>Gazebo/Black</material>
+        <mu1 value="0.001"/>
+        <mu2 value="0.001"/>
+    </gazebo>
 </robot>

Commit message: Adding Slam with slam-toolbox

File: description/robot_core.xacro (robot description, xacro)
@@ -17,7 +17,5 @@
         <color rgba="0 0 0 1"/>
     </material>
-    <link name="base_link">
-    </link>
-    <!-- CHASSIS -->
+    <!-- PROPERTY -->
     <xacro:property name="longueur_robot" value="0.25" />
     <xacro:property name="largeur_robot" value="0.15" />
@@ -25,4 +23,22 @@
     <xacro:property name="distance_cir" value="0.07836" />
     <xacro:property name="masse_robot" value="0.5" />
+    <xacro:property name="distance_cir_roue" value="0.1" />
+    <xacro:property name="longueur_roue" value="0.03" />
+    <xacro:property name="diametre_roue" value="0.065" />
+    <xacro:property name="masse_roue" value="0.1" />
+    <xacro:property name="diametre_caster" value="${diametre_roue}" />
+    <xacro:property name="distance_caster" value="0.20" />
+    <xacro:property name="masse_caster" value="0.1" />
+    <!-- BASE LINK -->
+    <link name="base_link"></link>
+    <!-- BASE LINK FOOTPRINT -->
+    <joint name="base_footprint_joint" type="fixed">
+        <parent link="base_link"/>
+        <child link="base_footprint"/>
+        <origin xyz="0 0 -${diametre_roue/2}" rpy="0 0 0"/>
+    </joint>
+    <link name="base_footprint">
+    </link>
+    <!-- CHASSIS -->
     <joint name="chassis_joint" type="fixed">
         <parent link="base_link"/>
@@ -52,8 +68,4 @@
     </gazebo>
     <!-- LEFT WHEEL -->
-    <xacro:property name="distance_cir_roue" value="0.1" />
-    <xacro:property name="longueur_roue" value="0.03" />
-    <xacro:property name="diametre_roue" value="0.065" />
-    <xacro:property name="masse_roue" value="0.1" />
     <joint name="left_wheel_joint" type="continuous">
         <parent link="base_link"/>
@@ -108,7 +120,4 @@
     </gazebo>
     <!-- CASTER WHEEL -->
-    <xacro:property name="diametre_caster" value="${diametre_roue}" />
-    <xacro:property name="distance_caster" value="0.20" />
-    <xacro:property name="masse_caster" value="0.1" />
     <joint name="caster_wheel_joint" type="fixed">
         <parent link="chassis"/>
