Commit message: Modify description file to match to real robot

File: description/camera.xacro (robot description, xacro)
@@ -1,12 +1,14 @@
 <?xml version="1.0"?>
 <robot xmlns:xacro="http://www.ros.org/wiki/xacro" >
-    <xacro:property name="longueur_camera" value="0.010" />
+    <xacro:property name="longueur_camera" value="0.020" />
     <xacro:property name="largeur_camera" value="0.03" />
     <xacro:property name="hauteur_camera" value="0.03" />
+    <xacro:property name="hauteur_base_camera" value="0.0985" />
     <xacro:property name="masse_camera" value="0.05" />
+    <xacro:property name="distance_camera" value="${0.190+(longueur_robot/2)}" />
     <joint name="camera_joint" type="fixed">
         <parent link="chassis"/>
         <child link="camera_link"/>
-        <origin xyz="${longueur_robot} 0 ${hauteur_robot/2}" rpy="0 0 0"/>
+        <origin xyz="${distance_camera} 0 ${hauteur_base_camera}" rpy="0 0 0"/>
     </joint>
     <link name="camera_link">

File: description/lidar.xacro (robot description, xacro)
@@ -1,12 +1,13 @@
 <?xml version="1.0"?>
 <robot xmlns:xacro="http://www.ros.org/wiki/xacro" >
-    <xacro:property name="distance_lidar" value="0.1" />
-    <xacro:property name="diametre_lidar" value="0.1" />
+    <xacro:property name="distance_lidar" value="0.217" />
+    <xacro:property name="diametre_lidar" value="0.068" />
     <xacro:property name="longueur_lidar" value="0.04" />
+    <xacro:property name="hauteur_lidar" value="0.169" />
     <xacro:property name="masse_lidar" value="0.1" />
     <joint name="laser_joint" type="fixed">
         <parent link="chassis"/>
         <child link="laser_frame"/>
-        <origin xyz="${distance_lidar} 0 ${hauteur_robot+(longueur_lidar/2)}" rpy="0 0 0"/>
+        <origin xyz="${distance_lidar} 0 ${hauteur_lidar}" rpy="0 0 0"/>
     </joint>
     <link name="laser_frame">

File: description/robot.urdf.xacro (robot description, xacro)
@@ -1,8 +1,14 @@
 <?xml version="1.0"?>
 <robot xmlns:xacro="http://www.ros.org/wiki/xacro"  name="robot">
+    <xacro:arg name="use_ros2_control" default="true"/>
+    <xacro:arg name="sim_mode" default="false"/>
     <xacro:include filename="robot_core.xacro" />
-    <!-- <xacro:include filename="gazebo_control.xacro"/> -->
     <xacro:include filename="lidar.xacro"/>
     <xacro:include filename="camera.xacro"/>
-    <xacro:include filename="ros2_control.xacro"/>
+    <xacro:if value="$(arg use_ros2_control)">
+        <xacro:include filename="ros2_control.xacro" />
+    </xacro:if>
+    <xacro:unless value="$(arg use_ros2_control)">
+        <xacro:include filename="gazebo_control.xacro" />
+    </xacro:unless>
 </robot>

File: description/robot_core.xacro (robot description, xacro)
@@ -18,15 +18,15 @@
     </material>
     <!-- PROPERTY -->
-    <xacro:property name="longueur_robot" value="0.25" />
-    <xacro:property name="largeur_robot" value="0.15" />
-    <xacro:property name="hauteur_robot" value="0.084" />
-    <xacro:property name="distance_cir" value="0.07836" />
-    <xacro:property name="masse_robot" value="0.5" />
-    <xacro:property name="distance_cir_roue" value="0.1" />
-    <xacro:property name="longueur_roue" value="0.03" />
-    <xacro:property name="diametre_roue" value="0.065" />
+    <xacro:property name="longueur_robot" value="0.308" />
+    <xacro:property name="largeur_robot" value="0.258" />
+    <xacro:property name="hauteur_robot" value="0.158" />
+    <xacro:property name="distance_cir" value="0.07" />
+    <xacro:property name="masse_robot" value="1" />
+    <xacro:property name="distance_cir_roue" value="${(largeur_robot/2)-longueur_roue}" />
+    <xacro:property name="longueur_roue" value="0.025" />
+    <xacro:property name="diametre_roue" value="0.068" />
     <xacro:property name="masse_roue" value="0.1" />
+    <xacro:property name="distance_caster" value="${longueur_robot-0.066}" />
     <xacro:property name="diametre_caster" value="${diametre_roue}" />
-    <xacro:property name="distance_caster" value="0.20" />
     <xacro:property name="masse_caster" value="0.1" />
     <!-- BASE LINK -->

File: description/ros2_control.xacro (robot description, xacro)
@@ -1,29 +1,66 @@
 <?xml version="1.0"?>
 <robot xmlns:xacro="http://www.ros.org/wiki/xacro">
-    <xacro:property name="vitesse_max_roue" value="10" />
-    <ros2_control name="GazeboSystem" type="system">
-        <hardware>
-            <plugin>gazebo_ros2_control/GazeboSystem</plugin>
-        </hardware>
-        <joint name="left_wheel_joint">
-            <command_interface name="velocity">
-                <param name="min">-${vitesse_max_roue}</param>
-                <param name="max">${vitesse_max_roue}</param>
-            </command_interface>
-            <state_interface name="position" />
-            <state_interface name="velocity" />
-        </joint>
-        <joint name="right_wheel_joint">
-            <command_interface name="velocity">
-                <param name="min">-${vitesse_max_roue}</param>
-                <param name="max">${vitesse_max_roue}</param>
-            </command_interface>
-            <state_interface name="velocity" />
-            <state_interface name="position" />
-        </joint>
-    </ros2_control>
+    <xacro:property name="vitesse_max_roue" value="5" />
+    <xacro:unless value="$(arg sim_mode)">
+        <ros2_control name="RealRobot" type="system">
+            <hardware>
+                <plugin>diffdrive_arduino/DiffDriveArduinoHardware</plugin>
+                <param name="left_wheel_name">left_wheel_joint</param>
+                <param name="right_wheel_name">right_wheel_joint</param>
+                <param name="loop_rate">30</param>
+                <param name="device">/dev/serial/by-path/pci-0000:06:00.4-usb-0:1:1.0</param>
+                <param name="baud_rate">57600</param>
+                <param name="timeout_ms">1000</param>
+                <param name="enc_counts_per_rev_left">3570</param>
+                <param name="enc_counts_per_rev_right">3476</param>
+                <param name="pid_p">20</param>
+                <param name="pid_d">12</param>
+                <param name="pid_i">0</param>
+                <param name="pid_o">50</param>
+            </hardware>
+            <joint name="left_wheel_joint">
+                <command_interface name="velocity">
+                    <param name="min">-${vitesse_max_roue}</param>
+                    <param name="max">${vitesse_max_roue}</param>
+                </command_interface>
+                <state_interface name="position" />
+                <state_interface name="velocity" />
+            </joint>
+            <joint name="right_wheel_joint">
+                <command_interface name="velocity">
+                    <param name="min">-${vitesse_max_roue}</param>
+                    <param name="max">${vitesse_max_roue}</param>
+                </command_interface>
+                <state_interface name="position" />
+                <state_interface name="velocity" />
+            </joint>
+        </ros2_control>
+    </xacro:unless>
+    <xacro:if value="$(arg sim_mode)">
+        <ros2_control name="GazeboSystem" type="system">
+            <hardware>
+                <plugin>gazebo_ros2_control/GazeboSystem</plugin>
+            </hardware>
+            <joint name="left_wheel_joint">
+                <command_interface name="velocity">
+                    <param name="min">-${vitesse_max_roue}</param>
+                    <param name="max">${vitesse_max_roue}</param>
+                </command_interface>
+                <state_interface name="position" />
+                <state_interface name="velocity" />
+            </joint>
+            <joint name="right_wheel_joint">
+                <command_interface name="velocity">
+                    <param name="min">-${vitesse_max_roue}</param>
+                    <param name="max">${vitesse_max_roue}</param>
+                </command_interface>
+                <state_interface name="velocity" />
+                <state_interface name="position" />
+            </joint>
+        </ros2_control>
+    </xacro:if>
     <gazebo>
         <plugin filename="libgazebo_ros2_control.so" name="gazebo_ros2_control">
-            <parameters>$(find my_robot)/params/my_controllers.yaml</parameters>
+            <parameters>$(find my_robot)/params/my_sim_controllers.yaml</parameters>
         </plugin>
     </gazebo>
