Commit message: Adding real robot files

File: description/robot.urdf.xacro (robot description, xacro)
@@ -3,4 +3,5 @@
     <xacro:arg name="use_ros2_control" default="true"/>
     <xacro:arg name="sim_mode" default="false"/>
+    <xacro:property name="PI" value="3.14159265359" />
     <xacro:include filename="robot_core.xacro" />
     <xacro:include filename="lidar.xacro"/>

File: description/ros2_control.xacro (robot description, xacro)
@@ -1,5 +1,5 @@
 <?xml version="1.0"?>
 <robot xmlns:xacro="http://www.ros.org/wiki/xacro">
-    <xacro:property name="vitesse_max_roue" value="5" />
+    <xacro:property name="vitesse_max_roue" value="2" />
     <xacro:unless value="$(arg sim_mode)">
         <ros2_control name="RealRobot" type="system">
@@ -9,9 +9,9 @@
                 <param name="right_wheel_name">right_wheel_joint</param>
                 <param name="loop_rate">30</param>
-                <param name="device">/dev/serial/by-path/pci-0000:06:00.4-usb-0:1:1.0</param>
+                <param name="device">/dev/serial/by-path/platform-fd500000.pcie-pci-0000:01:00.0-usb-0:1.2:1.0</param>
                 <param name="baud_rate">57600</param>
                 <param name="timeout_ms">1000</param>
-                <param name="enc_counts_per_rev_left">3570</param>
-                <param name="enc_counts_per_rev_right">3476</param>
+                <param name="enc_counts_per_rev_left">3572</param>
+                <param name="enc_counts_per_rev_right">3472</param>
                 <param name="pid_p">20</param>
                 <param name="pid_d">12</param>
